Commit message: meshes and urdf

File: urdf/tr1.urdf (robot description, URDF)
Before this commit: robot tr1, 2 links, 1 joints
Links:
- removed link riserbase_link
- added link wheel_link; visual box size=0.225 0.471 0.339
- link base_link: geometry visual mesh filename=package://tr1_description/meshes/base.dae
Joints:
- removed joint base_to_riserbase
- added joint base_to_wheel: type fixed, parent base_link, child wheel_link, origin xyz=0 0.2 0.1115

Commit message: body dae to urdf

File: urdf/tr1.urdf (robot description, URDF)
Before this commit: robot tr1, 2 links, 1 joints
Links:
- removed link wheel_link
- added link body_link; visual mesh filename=package://tr1_description/meshes/body.dae scale=0.1 0.1 0.1
- link base_link: geometry visual mesh filename=package://tr1_description/meshes/base.dae scale=0.1 0.1 0.1
Joints:
- removed joint base_to_wheel
- added joint base_to_body: type prismatic, parent base_link, child body_link, origin xyz=0 0 0.8 rpy=0 0 0, limit lower=0 upper=150 effort=1000.0 velocity=0.5

Commit message: urdf creation

File: urdf/tr1.urdf (robot description, URDF)
Before this commit: robot tr1, 2 links, 1 joints
Links:
- added link head_link; visual mesh filename=package://tr1_description/meshes/head.dae scale=0.1 0.1 0.1
- added link neck_base_link; visual mesh filename=package://tr1_description/meshes/neck_base.dae scale=0.1 0.1 0.1
- added link neck_link; visual mesh filename=package://tr1_description/meshes/neck.dae scale=0.1 0.1 0.1
Joints:
- added joint body_to_neck_base: type fixed, parent body_link, child neck_base_link, origin xyz=0 0 0.4 rpy=0 0 0
- added joint neck_base_to_neck: type revolute, parent neck_base_link, child neck_link, origin xyz=0 0 0.033 rpy=0 0 0, axis 0 0 1, limit lower=-3.1415 upper=3.1415 effort=1.0 velocity=0.5
- added joint neck_to_head: type revolute, parent neck_link, child head_link, origin xyz=0 0.090789 0.09 rpy=0 0 0, axis 1 0 0, limit lower=-0.9 upper=0.4 effort=1.0 velocity=0.5
- joint base_to_body: axis (none) -> 0 0 1; limit lower=0 upper=150 effort=1000.0 velocity=0.5 -> lower=0 upper=0.300 effort=1000.0 velocity=0.0001; origin xyz=0 0 0.8 rpy=0 0 0 -> xyz=0 0 0.76 rpy=0 0 0

Commit message: urdf measurements

File: urdf/tr1.urdf (robot description, URDF)
Before this commit: robot tr1, 5 links, 4 joints
Links:
- added link arm1_link; visual mesh filename=package://tr1_description/meshes/arm1.dae scale=0.1 0.1 0.1
Joints:
- added joint body_to_arm1: type fixed, parent body_link, child arm1_link, origin xyz=0.155887 0.026656 0.2075 rpy=0 0 0
- joint base_to_body: origin xyz=0 0 0.76 rpy=0 0 0 -> xyz=0 0 0.7955 rpy=0 0 0

Commit message: urdf mesh and link measurements

File: urdf/tr1.urdf (robot description, URDF)
Before this commit: robot tr1, 6 links, 5 joints
Joints:
- joint body_to_arm1: origin xyz=0.155887 0.026656 0.2075 rpy=0 0 0 -> xyz=0.155887 0.026656 0.2075 rpy=0 0 0.261799
- joint body_to_neck_base: origin xyz=0 0 0.4 rpy=0 0 0 -> xyz=0 0 0.365 rpy=0 0 0

Commit message: measurements

File: urdf/tr1.urdf (robot description, URDF)
Before this commit: robot tr1, 6 links, 5 joints
Links:
- added link arm2_link; visual mesh filename=package://tr1_description/meshes/arm2.dae scale=0.1 0.1 0.1
- added link arm3_link; visual mesh filename=package://tr1_description/meshes/arm3.dae scale=0.1 0.1 0.1
- added link arm4_link; visual mesh filename=package://tr1_description/meshes/arm4.dae scale=0.1 0.1 0.1
- added link arm5_link; visual mesh filename=package://tr1_description/meshes/arm5.dae scale=0.1 0.1 0.1
- added link arm6_link; visual mesh filename=package://tr1_description/meshes/arm6.dae scale=0.1 0.1 0.1
- added link arm7_link; visual mesh filename=package://tr1_description/meshes/arm7.dae scale=0.1 0.1 0.1
- added link arm8_link; visual mesh filename=package://tr1_description/meshes/arm8.dae scale=0.1 0.1 0.1
Joints:
- added joint arm1_to_arm2: type fixed, parent arm1_link, child arm2_link, origin xyz=0 0.139238 0 rpy=0 0 0
- added joint arm2_to_arm3: type fixed, parent arm2_link, child arm3_link, origin xyz=0 0 0 rpy=0 0 0
- added joint arm3_to_arm4: type fixed, parent arm3_link, child arm4_link, origin xyz=0 0 0 rpy=0 0 0
- added joint arm4_to_arm5: type fixed, parent arm4_link, child arm5_link, origin xyz=0 0 0 rpy=0 0 0
- added joint arm5_to_arm6: type fixed, parent arm5_link, child arm6_link, origin xyz=0 0 0 rpy=0 0 0
- added joint arm6_to_arm7: type fixed, parent arm6_link, child arm7_link, origin xyz=0 0 0 rpy=0 0 0
- added joint arm7_to_arm8: type fixed, parent arm7_link, child arm8_link, origin xyz=0 0 0 rpy=0 0 0

Commit message: measurements

File: urdf/tr1.urdf (robot description, URDF)
Before this commit: robot tr1, 13 links, 12 joints
Joints:
- joint arm1_to_arm2: origin xyz=0 0.139238 0 rpy=0 0 0 -> xyz=0 0 0 rpy=0 0 0
- joint arm2_to_arm3: origin xyz=0 0 0 rpy=0 0 0 -> xyz=0 0.139238 0 rpy=0 0 0

Commit message: measurements

File: urdf/tr1.urdf (robot description, URDF)
Before this commit: robot tr1, 13 links, 12 joints
Joints:
- joint arm1_to_arm2: axis (none) -> 0 0 1; limit (none) -> lower=-1 upper=1.5708 effort=1.0 velocity=0.5; origin xyz=0 0 0 rpy=0 0 0 -> xyz=0 0 -0.007 rpy=0 0 0; type fixed -> revolute
- joint arm2_to_arm3: axis (none) -> 0 1 0; limit (none) -> lower=-1 upper=1.5708 effort=1.0 velocity=0.5; origin xyz=0 0.139238 0 rpy=0 0 0 -> xyz=0.139238 0 0 rpy=0 0 0; type fixed -> revolute
- joint body_to_arm1: origin xyz=0.155887 0.026656 0.2075 rpy=0 0 0.261799 -> xyz=0.184864 0.034420 0.2075 rpy=0 0 0.261799
- joint body_to_neck_base: origin xyz=0 0 0.365 rpy=0 0 0 -> xyz=0 -0.017 0.365 rpy=0 0 0

Commit message: design wip :

File: urdf/tr1.urdf (robot description, URDF)
Before this commit: robot tr1, 13 links, 12 joints
Joints:
- joint arm3_to_arm4: axis (none) -> 1 0 0; limit (none) -> lower=-3.1415 upper=3.1415 effort=1.0 velocity=0.5; origin xyz=0 0 0 rpy=0 0 0 -> xyz=0.238827 0 0 rpy=0 0 0; type fixed -> revolute
- joint arm4_to_arm5: axis (none) -> 0 1 0; limit (none) -> lower=-3.1415 upper=3.1415 effort=1.0 velocity=0.5; origin xyz=0 0 0 rpy=0 0 0 -> xyz=0.145 0 0 rpy=0 0 0; type fixed -> revolute
- joint arm5_to_arm6: axis (none) -> 1 0 0; limit (none) -> lower=-3.1415 upper=3.1415 effort=1.0 velocity=0.5; origin xyz=0 0 0 rpy=0 0 0 -> xyz=0.230643 0 0 rpy=0 0 0; type fixed -> revolute
- joint arm6_to_arm7: origin xyz=0 0 0 rpy=0 0 0 -> xyz=0.165 0 0 rpy=0 0 0

Commit message: measurements

File: urdf/tr1.urdf (robot description, URDF)
Before this commit: robot tr1, 13 links, 12 joints
Links:
- added link gripper1_link; visual mesh filename=package://tr1_description/meshes/gripper1.dae scale=0.1 0.1 0.1
Joints:
- added joint arm8_to_gripper1: type fixed, parent arm8_link, child gripper1_link, origin xyz=0.04619 0 0 rpy=0 0 0
- joint arm6_to_arm7: axis (none) -> 0 1 0; limit (none) -> lower=-3.1415 upper=3.1415 effort=1.0 velocity=0.5; type fixed -> revolute
- joint arm7_to_arm8: axis (none) -> 1 0 0; limit (none) -> lower=-3.1415 upper=3.1415 effort=1.0 velocity=0.5; origin xyz=0 0 0 rpy=0 0 0 -> xyz=0.045311 0 0 rpy=0 0 0; type fixed -> revolute
- joint body_to_arm1: origin xyz=0.184864 0.034420 0.2075 rpy=0 0 0.261799 -> xyz=0.184864 0.034420 0.20575 rpy=0 0 0.261799

Commit message: measurements

File: urdf/tr1.urdf (robot description, URDF)
Before this commit: robot tr1, 14 links, 13 joints
Links:
- added link gripper2_link; visual mesh filename=package://tr1_description/meshes/gripper2.dae scale=0.1 0.1 0.1
- added link gripper3_link; visual mesh filename=package://tr1_description/meshes/gripper3.dae scale=0.1 0.1 0.1
- added link gripper4l_link; visual mesh filename=package://tr1_description/meshes/gripper4.dae scale=0.1 0.1 0.1
- added link gripper4r_link; visual mesh filename=package://tr1_description/meshes/gripper4.dae scale=0.1 0.1 0.1
- added link gripper5_link; visual mesh filename=package://tr1_description/meshes/gripper5.dae scale=0.1 0.1 0.1
- added link gripper6_link; visual mesh filename=package://tr1_description/meshes/gripper6.dae scale=0.1 0.1 0.1
Joints:
- added joint gripper1_to_gripper2: type fixed, parent gripper1_link, child gripper2_link, origin xyz=0.024 -0.014 0 rpy=0 0 -1.5708
- added joint gripper1_to_gripper3: type fixed, parent gripper1_link, child gripper3_link, origin xyz=0.024 0.014 0 rpy=0 0 1.5708
- added joint gripper1_to_gripper4l: type fixed, parent gripper1_link, child gripper4l_link, origin xyz=0.044 0.007 0 rpy=0 0 -1.5708
- added joint gripper1_to_gripper4r: type fixed, parent gripper1_link, child gripper4r_link, origin xyz=0.044 -0.007 0 rpy=0 0 1.5708
- added joint gripper2_to_gripper6: type fixed, parent gripper2_link, child gripper6_link, origin xyz=0.040 0 0 rpy=0 0 0
- added joint gripper3_to_gripper5: type fixed, parent gripper3_link, child gripper5_link, origin xyz=0.040 0 0 rpy=0 0 0

Commit message: measurements

File: urdf/tr1.urdf (robot description, URDF)
Before this commit: robot tr1, 20 links, 19 joints
Joints:
- removed joint gripper1_to_gripper2
- added joint gripper: type revolute, parent gripper1_link, child gripper2_link, origin xyz=0.024 -0.014 0 rpy=0 0 -1.5708, axis 0 0 1, limit lower=0 upper=1.5708 effort=1.0 velocity=0.5
- joint arm2_to_arm3: limit lower=-1 upper=1.5708 effort=1.0 velocity=0.5 -> lower=-1.5708 upper=1.5708 effort=1.0 velocity=0.5
- joint arm4_to_arm5: limit lower=-3.1415 upper=3.1415 effort=1.0 velocity=0.5 -> lower=-1.75 upper=1.75 effort=1.0 velocity=0.5
- joint arm6_to_arm7: limit lower=-3.1415 upper=3.1415 effort=1.0 velocity=0.5 -> lower=-1.75 upper=1.75 effort=1.0 velocity=0.5
- joint arm7_to_arm8: limit lower=-3.1415 upper=3.1415 effort=1.0 velocity=0.5 -> lower=-2 upper=2 effort=1.0 velocity=0.5
- joint gripper1_to_gripper3: axis (none) -> 0 0 1; limit (none) -> lower=-3.1415 upper=3.1415 effort=1.0 velocity=0.5; mimic (none) -> joint=gripper multiplier=-1 offset=0; type fixed -> revolute
- joint gripper1_to_gripper4l: axis (none) -> 0 0 1; limit (none) -> lower=-3.1415 upper=3.1415 effort=1.0 velocity=0.5; mimic (none) -> joint=gripper multiplier=-1 offset=0; type fixed -> revolute
- joint gripper1_to_gripper4r: axis (none) -> 0 0 1; limit (none) -> lower=-3.1415 upper=3.1415 effort=1.0 velocity=0.5; mimic (none) -> joint=gripper multiplier=1 offset=0; type fixed -> revolute
- joint gripper2_to_gripper6: axis (none) -> 0 0 1; limit (none) -> lower=-3.1415 upper=3.1415 effort=1.0 velocity=0.5; mimic (none) -> joint=gripper multiplier=-1 offset=0; type fixed -> revolute
- joint gripper3_to_gripper5: axis (none) -> 0 0 1; limit (none) -> lower=-3.1415 upper=3.1415 effort=1.0 velocity=0.5; mimic (none) -> joint=gripper multiplier=1 offset=0; type fixed -> revolute

Commit message: urdf rework

File: urdf/tr1.urdf (robot description, URDF)
Before this commit: robot tr1, 20 links, 19 joints
Links:
- added link wheel1_link; visual mesh filename=package://tr1_description/meshes/dae/wheel.dae scale=0.001 0.001 0.001
- added link wheel2_link; visual mesh filename=package://tr1_description/meshes/dae/wheel.dae scale=0.001 0.001 0.001
- added link wheel3_link; visual mesh filename=package://tr1_description/meshes/dae/wheel.dae scale=0.001 0.001 0.001
- added link wheel4_link; visual mesh filename=package://tr1_description/meshes/dae/wheel.dae scale=0.001 0.001 0.001
- link arm1_link: geometry visual mesh filename=package://tr1_description/meshes/dae/arm1.dae scale=0.001 0.001 0.001
- link arm2_link: geometry visual mesh filename=package://tr1_description/meshes/dae/arm2.dae scale=0.001 0.001 0.001
- link arm3_link: geometry visual mesh filename=package://tr1_description/meshes/dae/arm3.dae scale=0.001 0.001 0.001
- link arm4_link: geometry visual mesh filename=package://tr1_description/meshes/dae/arm4.dae scale=0.001 0.001 0.001
- link arm5_link: geometry visual mesh filename=package://tr1_description/meshes/dae/arm5.dae scale=0.001 0.001 0.001
- link arm6_link: geometry visual mesh filename=package://tr1_description/meshes/dae/arm6.dae scale=0.001 0.001 0.001
- link arm7_link: geometry visual mesh filename=package://tr1_description/meshes/dae/arm7.dae scale=0.001 0.001 0.001
- link arm8_link: geometry visual mesh filename=package://tr1_description/meshes/dae/arm8.dae scale=0.001 0.001 0.001
- link base_link: geometry visual mesh filename=package://tr1_description/meshes/dae/base.dae scale=0.001 0.001 0.001
- link body_link: geometry visual mesh filename=package://tr1_description/meshes/dae/body.dae scale=0.001 0.001 0.001
- link gripper1_link: geometry visual mesh filename=package://tr1_description/meshes/dae/gripper1.dae scale=0.001 0.001 0.001
- link gripper2_link: geometry visual mesh filename=package://tr1_description/meshes/dae/gripper2.dae scale=0.001 0.001 0.001
- link gripper3_link: geometry visual mesh filename=package://tr1_description/meshes/dae/gripper3.dae scale=0.001 0.001 0.001
- link gripper4l_link: geometry visual mesh filename=package://tr1_description/meshes/dae/gripper4.dae scale=0.001 0.001 0.001
- link gripper4r_link: geometry visual mesh filename=package://tr1_description/meshes/dae/gripper4.dae scale=0.001 0.001 0.001
- link gripper5_link: geometry visual mesh filename=package://tr1_description/meshes/dae/gripper5.dae scale=0.001 0.001 0.001
- link gripper6_link: geometry visual mesh filename=package://tr1_description/meshes/dae/gripper6.dae scale=0.001 0.001 0.001
- link head_link: geometry visual mesh filename=package://tr1_description/meshes/dae/head.dae scale=0.001 0.001 0.001
- link neck_base_link: geometry visual mesh filename=package://tr1_description/meshes/dae/neck_base.dae scale=0.001 0.001 0.001
- link neck_link: geometry visual mesh filename=package://tr1_description/meshes/dae/neck.dae scale=0.001 0.001 0.001
Joints:
- added joint base_to_wheel1: type continuous, parent base_link, child wheel1_link, origin xyz=-0.293310 0.417810 -0.0725 rpy=0 0 0.785398, axis 0 1 0
- added joint base_to_wheel2: type continuous, parent base_link, child wheel2_link, origin xyz=0.293310 0.417810 -0.0725 rpy=0 0 -0.785398, axis 0 1 0
- added joint base_to_wheel3: type continuous, parent base_link, child wheel3_link, origin xyz=0.293310 -0.168810 -0.0725 rpy=0 0 -2.35619449019, axis 0 1 0
- added joint base_to_wheel4: type continuous, parent base_link, child wheel4_link, origin xyz=-0.293310 -0.168810 -0.0725 rpy=0 0 2.356194490191, axis 0 1 0
- joint arm1_to_arm2: origin xyz=0 0 -0.007 rpy=0 0 0 -> xyz=0 0 -0.007
- joint arm2_to_arm3: origin xyz=0.139238 0 0 rpy=0 0 0 -> xyz=0.139238 0 0
- joint arm3_to_arm4: origin xyz=0.238827 0 0 rpy=0 0 0 -> xyz=0.238827 0 0
- joint arm4_to_arm5: origin xyz=0.145 0 0 rpy=0 0 0 -> xyz=0.145 0 0
- joint arm5_to_arm6: origin xyz=0.230643 0 0 rpy=0 0 0 -> xyz=0.230643 0 0
- joint arm6_to_arm7: origin xyz=0.165 0 0 rpy=0 0 0 -> xyz=0.165 0 0
- joint arm7_to_arm8: origin xyz=0.045311 0 0 rpy=0 0 0 -> xyz=0.045311 0 0
- joint arm8_to_gripper1: origin xyz=0.04619 0 0 rpy=0 0 0 -> xyz=0.04619 0 0
- joint base_to_body: origin xyz=0 0 0.7955 rpy=0 0 0 -> xyz=0 0 0.7955
- joint body_to_neck_base: origin xyz=0 -0.017 0.365 rpy=0 0 0 -> xyz=0 -0.017 0.365
- joint gripper2_to_gripper6: origin xyz=0.040 0 0 rpy=0 0 0 -> xyz=0.040 0 0
- joint gripper3_to_gripper5: origin xyz=0.040 0 0 rpy=0 0 0 -> xyz=0.040 0 0
- joint neck_base_to_neck: origin xyz=0 0 0.033 rpy=0 0 0 -> xyz=0 0 0.033
- joint neck_to_head: origin xyz=0 0.090789 0.09 rpy=0 0 0 -> xyz=0 0.090789 0.09
