Commit message: second arm added

File: urdf/tr1.urdf (robot description, URDF)
Before this commit: robot tr1, 24 links, 23 joints
Links:
- removed link arm1_link
- removed link arm2_link
- removed link arm3_link
- removed link arm4_link
- removed link arm5_link
- removed link arm6_link
- removed link arm7_link
- removed link arm8_link
- removed link gripper1_link
- removed link gripper2_link
- removed link gripper3_link
- removed link gripper4l_link
- removed link gripper4r_link
- removed link gripper5_link
- removed link gripper6_link
- added link left_arm1_link; visual mesh filename=package://tr1_description/meshes/dae/arm1.dae scale=0.001 0.001 0.001
- added link left_arm2_link; visual mesh filename=package://tr1_description/meshes/dae/arm2.dae scale=0.001 0.001 0.001
- added link left_arm3_link; visual mesh filename=package://tr1_description/meshes/dae/arm3.dae scale=0.001 0.001 0.001
- added link left_arm4_link; visual mesh filename=package://tr1_description/meshes/dae/arm4.dae scale=0.001 0.001 0.001
- added link left_arm5_link; visual mesh filename=package://tr1_description/meshes/dae/arm5.dae scale=0.001 0.001 0.001
- added link left_arm6_link; visual mesh filename=package://tr1_description/meshes/dae/arm6.dae scale=0.001 0.001 0.001
- added link left_arm7_link; visual mesh filename=package://tr1_description/meshes/dae/arm7.dae scale=0.001 0.001 0.001
- added link left_arm8_link; visual mesh filename=package://tr1_description/meshes/dae/arm8.dae scale=0.001 0.001 0.001
- added link left_gripper1_link; visual mesh filename=package://tr1_description/meshes/dae/gripper1.dae scale=0.001 0.001 0.001
- added link left_gripper2_link; visual mesh filename=package://tr1_description/meshes/dae/gripper2.dae scale=0.001 0.001 0.001
- added link left_gripper3_link; visual mesh filename=package://tr1_description/meshes/dae/gripper3.dae scale=0.001 0.001 0.001
- added link left_gripper4l_link; visual mesh filename=package://tr1_description/meshes/dae/gripper4.dae scale=0.001 0.001 0.001
- added link left_gripper4r_link; visual mesh filename=package://tr1_description/meshes/dae/gripper4.dae scale=0.001 0.001 0.001
- added link left_gripper5_link; visual mesh filename=package://tr1_description/meshes/dae/gripper5.dae scale=0.001 0.001 0.001
- added link left_gripper6_link; visual mesh filename=package://tr1_description/meshes/dae/gripper6.dae scale=0.001 0.001 0.001
- added link right_arm1_link; visual mesh filename=package://tr1_description/meshes/dae/arm1.dae scale=0.001 0.001 0.001
- added link right_arm2_link; visual mesh filename=package://tr1_description/meshes/dae/arm2.dae scale=0.001 0.001 0.001
- added link right_arm3_link; visual mesh filename=package://tr1_description/meshes/dae/arm3.dae scale=0.001 0.001 0.001
- added link right_arm4_link; visual mesh filename=package://tr1_description/meshes/dae/arm4.dae scale=0.001 0.001 0.001
- added link right_arm5_link; visual mesh filename=package://tr1_description/meshes/dae/arm5.dae scale=0.001 0.001 0.001
- added link right_arm6_link; visual mesh filename=package://tr1_description/meshes/dae/arm6.dae scale=0.001 0.001 0.001
- added link right_arm7_link; visual mesh filename=package://tr1_description/meshes/dae/arm7.dae scale=0.001 0.001 0.001
- added link right_arm8_link; visual mesh filename=package://tr1_description/meshes/dae/arm8.dae scale=0.001 0.001 0.001
- added link right_gripper1_link; visual mesh filename=package://tr1_description/meshes/dae/gripper1.dae scale=0.001 0.001 0.001
- added link right_gripper2_link; visual mesh filename=package://tr1_description/meshes/dae/gripper2.dae scale=0.001 0.001 0.001
- added link right_gripper3_link; visual mesh filename=package://tr1_description/meshes/dae/gripper3.dae scale=0.001 0.001 0.001
- added link right_gripper4l_link; visual mesh filename=package://tr1_description/meshes/dae/gripper4.dae scale=0.001 0.001 0.001
- added link right_gripper4r_link; visual mesh filename=package://tr1_description/meshes/dae/gripper4.dae scale=0.001 0.001 0.001
- added link right_gripper5_link; visual mesh filename=package://tr1_description/meshes/dae/gripper5.dae scale=0.001 0.001 0.001
- added link right_gripper6_link; visual mesh filename=package://tr1_description/meshes/dae/gripper6.dae scale=0.001 0.001 0.001
Joints:
- removed joint arm1_to_arm2
- removed joint arm2_to_arm3
- removed joint arm3_to_arm4
- removed joint arm4_to_arm5
- removed joint arm5_to_arm6
- removed joint arm6_to_arm7
- removed joint arm7_to_arm8
- removed joint arm8_to_gripper1
- removed joint body_to_arm1
- removed joint gripper
- removed joint gripper1_to_gripper3
- removed joint gripper1_to_gripper4l
- removed joint gripper1_to_gripper4r
- removed joint gripper2_to_gripper6
- removed joint gripper3_to_gripper5
- added joint body_to_left_arm1: type fixed, parent body_link, child left_arm1_link, origin xyz=-0.184864 0.034420 0.20575 rpy=0 0 2.87979
- added joint body_to_right_arm1: type fixed, parent body_link, child right_arm1_link, origin xyz=0.184864 0.034420 0.20575 rpy=0 0 0.261799
- added joint left_arm1_to_left_arm2: type revolute, parent left_arm1_link, child left_arm2_link, origin xyz=0 0 -0.007, axis 0 0 1, limit lower=-1.5708 upper=1 effort=1.0 velocity=0.5
- added joint left_arm2_to_left_arm3: type revolute, parent left_arm2_link, child left_arm3_link, origin xyz=0.139238 0 0, axis 0 1 0, limit lower=-1.5708 upper=1.5708 effort=1.0 velocity=0.5
- added joint left_arm3_to_left_arm4: type revolute, parent left_arm3_link, child left_arm4_link, origin xyz=0.238827 0 0, axis 1 0 0, limit lower=-3.1415 upper=3.1415 effort=1.0 velocity=0.5
- added joint left_arm4_to_left_arm5: type revolute, parent left_arm4_link, child left_arm5_link, origin xyz=0.145 0 0, axis 0 1 0, limit lower=-1.75 upper=1.75 effort=1.0 velocity=0.5
- added joint left_arm5_to_left_arm6: type revolute, parent left_arm5_link, child left_arm6_link, origin xyz=0.230643 0 0, axis 1 0 0, limit lower=-3.1415 upper=3.1415 effort=1.0 velocity=0.5
- added joint left_arm6_to_left_arm7: type revolute, parent left_arm6_link, child left_arm7_link, origin xyz=0.165 0 0, axis 0 1 0, limit lower=-1.75 upper=1.75 effort=1.0 velocity=0.5
- added joint left_arm7_to_left_arm8: type revolute, parent left_arm7_link, child left_arm8_link, origin xyz=0.045311 0 0, axis 1 0 0, limit lower=-2 upper=2 effort=1.0 velocity=0.5
- added joint left_arm8_to_left_gripper1: type fixed, parent left_arm8_link, child left_gripper1_link, origin xyz=0.04619 0 0
- added joint left_gripper: type revolute, parent left_gripper1_link, child left_gripper2_link, origin xyz=0.024 -0.014 0 rpy=0 0 -1.5708, axis 0 0 1, limit lower=0 upper=1.5708 effort=1.0 velocity=0.5
- added joint left_gripper1_to_left_gripper3: type revolute, parent left_gripper1_link, child left_gripper3_link, origin xyz=0.024 0.014 0 rpy=0 0 1.5708, axis 0 0 1, limit lower=-3.1415 upper=3.1415 effort=1.0 velocity=0.5, mimic joint=left_gripper multiplier=-1 offset=0
- added joint left_gripper1_to_left_gripper4l: type revolute, parent left_gripper1_link, child left_gripper4l_link, origin xyz=0.044 0.007 0 rpy=0 0 -1.5708, axis 0 0 1, limit lower=-3.1415 upper=3.1415 effort=1.0 velocity=0.5, mimic joint=left_gripper multiplier=-1 offset=0
- added joint left_gripper1_to_left_gripper4r: type revolute, parent left_gripper1_link, child left_gripper4r_link, origin xyz=0.044 -0.007 0 rpy=0 0 1.5708, axis 0 0 1, limit lower=-3.1415 upper=3.1415 effort=1.0 velocity=0.5, mimic joint=left_gripper multiplier=1 offset=0
- added joint left_gripper2_to_left_gripper6: type revolute, parent left_gripper2_link, child left_gripper6_link, origin xyz=0.040 0 0, axis 0 0 1, limit lower=-3.1415 upper=3.1415 effort=1.0 velocity=0.5, mimic joint=left_gripper multiplier=-1 offset=0
- added joint left_gripper3_to_left_gripper5: type revolute, parent left_gripper3_link, child left_gripper5_link, origin xyz=0.040 0 0, axis 0 0 1, limit lower=-3.1415 upper=3.1415 effort=1.0 velocity=0.5, mimic joint=left_gripper multiplier=1 offset=0
- added joint right_arm1_to_right_arm2: type revolute, parent right_arm1_link, child right_arm2_link, origin xyz=0 0 -0.007, axis 0 0 1, limit lower=-1 upper=1.5708 effort=1.0 velocity=0.5
- added joint right_arm2_to_right_arm3: type revolute, parent right_arm2_link, child right_arm3_link, origin xyz=0.139238 0 0, axis 0 1 0, limit lower=-1.5708 upper=1.5708 effort=1.0 velocity=0.5
- added joint right_arm3_to_right_arm4: type revolute, parent right_arm3_link, child right_arm4_link, origin xyz=0.238827 0 0, axis 1 0 0, limit lower=-3.1415 upper=3.1415 effort=1.0 velocity=0.5
- added joint right_arm4_to_right_arm5: type revolute, parent right_arm4_link, child right_arm5_link, origin xyz=0.145 0 0, axis 0 1 0, limit lower=-1.75 upper=1.75 effort=1.0 velocity=0.5
- added joint right_arm5_to_right_arm6: type revolute, parent right_arm5_link, child right_arm6_link, origin xyz=0.230643 0 0, axis 1 0 0, limit lower=-3.1415 upper=3.1415 effort=1.0 velocity=0.5
- added joint right_arm6_to_right_arm7: type revolute, parent right_arm6_link, child right_arm7_link, origin xyz=0.165 0 0, axis 0 1 0, limit lower=-1.75 upper=1.75 effort=1.0 velocity=0.5
- added joint right_arm7_to_right_arm8: type revolute, parent right_arm7_link, child right_arm8_link, origin xyz=0.045311 0 0, axis 1 0 0, limit lower=-2 upper=2 effort=1.0 velocity=0.5
- added joint right_arm8_to_right_gripper1: type fixed, parent right_arm8_link, child right_gripper1_link, origin xyz=0.04619 0 0
- added joint right_gripper: type revolute, parent right_gripper1_link, child right_gripper2_link, origin xyz=0.024 -0.014 0 rpy=0 0 -1.5708, axis 0 0 1, limit lower=0 upper=1.5708 effort=1.0 velocity=0.5
- added joint right_gripper1_to_right_gripper3: type revolute, parent right_gripper1_link, child right_gripper3_link, origin xyz=0.024 0.014 0 rpy=0 0 1.5708, axis 0 0 1, limit lower=-3.1415 upper=3.1415 effort=1.0 velocity=0.5, mimic joint=right_gripper multiplier=-1 offset=0
- added joint right_gripper1_to_right_gripper4l: type revolute, parent right_gripper1_link, child right_gripper4l_link, origin xyz=0.044 0.007 0 rpy=0 0 -1.5708, axis 0 0 1, limit lower=-3.1415 upper=3.1415 effort=1.0 velocity=0.5, mimic joint=right_gripper multiplier=-1 offset=0
- added joint right_gripper1_to_right_gripper4r: type revolute, parent right_gripper1_link, child right_gripper4r_link, origin xyz=0.044 -0.007 0 rpy=0 0 1.5708, axis 0 0 1, limit lower=-3.1415 upper=3.1415 effort=1.0 velocity=0.5, mimic joint=right_gripper multiplier=1 offset=0
- added joint right_gripper2_to_right_gripper6: type revolute, parent right_gripper2_link, child right_gripper6_link, origin xyz=0.040 0 0, axis 0 0 1, limit lower=-3.1415 upper=3.1415 effort=1.0 velocity=0.5, mimic joint=right_gripper multiplier=-1 offset=0
- added joint right_gripper3_to_right_gripper5: type revolute, parent right_gripper3_link, child right_gripper5_link, origin xyz=0.040 0 0, axis 0 0 1, limit lower=-3.1415 upper=3.1415 effort=1.0 velocity=0.5, mimic joint=right_gripper multiplier=1 offset=0

Commit message: arm renaming

File: urdf/tr1.urdf (robot description, URDF)
Before this commit: robot tr1, 39 links, 38 joints
Joints:
- removed joint right_arm1_to_right_arm2
- removed joint right_arm2_to_right_arm3
- removed joint right_arm3_to_right_arm4
- removed joint right_arm4_to_right_arm5
- removed joint right_arm5_to_right_arm6
- removed joint right_arm6_to_right_arm7
- removed joint right_arm7_to_right_arm8
- removed joint right_gripper
- added joint JointRightElbowFlex: type revolute, parent right_arm4_link, child right_arm5_link, origin xyz=0.145 0 0, axis 0 1 0, limit lower=-1.75 upper=1.75 effort=1.0 velocity=0.5
- added joint JointRightForearmRoll: type revolute, parent right_arm5_link, child right_arm6_link, origin xyz=0.230643 0 0, axis 1 0 0, limit lower=-3.1415 upper=3.1415 effort=1.0 velocity=0.5
- added joint JointRightGripper: type revolute, parent right_gripper1_link, child right_gripper2_link, origin xyz=0.024 -0.014 0 rpy=0 0 -1.5708, axis 0 0 1, limit lower=0 upper=1.5708 effort=1.0 velocity=0.5
- added joint JointRightShoulderPan: type revolute, parent right_arm1_link, child right_arm2_link, origin xyz=0 0 -0.007, axis 0 0 1, limit lower=-1 upper=1.5708 effort=1.0 velocity=0.5
- added joint JointRightShoulderTilt: type revolute, parent right_arm2_link, child right_arm3_link, origin xyz=0.139238 0 0, axis 0 1 0, limit lower=-1.5708 upper=1.5708 effort=1.0 velocity=0.5
- added joint JointRightUpperArmRoll: type revolute, parent right_arm3_link, child right_arm4_link, origin xyz=0.238827 0 0, axis 1 0 0, limit lower=-3.1415 upper=3.1415 effort=1.0 velocity=0.5
- added joint JointRightWristFlex: type revolute, parent right_arm6_link, child right_arm7_link, origin xyz=0.165 0 0, axis 0 1 0, limit lower=-1.75 upper=1.75 effort=1.0 velocity=0.5
- added joint JointRightWristRoll: type revolute, parent right_arm7_link, child right_arm8_link, origin xyz=0.045311 0 0, axis 1 0 0, limit lower=-2 upper=2 effort=1.0 velocity=0.5
- joint right_gripper1_to_right_gripper3: mimic joint=right_gripper multiplier=-1 offset=0 -> joint=JointRightGripper multiplier=-1 offset=0
- joint right_gripper1_to_right_gripper4l: mimic joint=right_gripper multiplier=-1 offset=0 -> joint=JointRightGripper multiplier=-1 offset=0
- joint right_gripper1_to_right_gripper4r: mimic joint=right_gripper multiplier=1 offset=0 -> joint=JointRightGripper multiplier=1 offset=0
- joint right_gripper2_to_right_gripper6: mimic joint=right_gripper multiplier=-1 offset=0 -> joint=JointRightGripper multiplier=-1 offset=0
- joint right_gripper3_to_right_gripper5: mimic joint=right_gripper multiplier=1 offset=0 -> joint=JointRightGripper multiplier=1 offset=0

Commit message: urdf and rviz launch

File: urdf/tr1.urdf (robot description, URDF)
Before this commit: robot tr1, 39 links, 38 joints
Joints:
- removed joint left_arm1_to_left_arm2
- removed joint left_arm2_to_left_arm3
- removed joint left_arm3_to_left_arm4
- removed joint left_arm4_to_left_arm5
- removed joint left_arm5_to_left_arm6
- removed joint left_arm6_to_left_arm7
- removed joint left_arm7_to_left_arm8
- removed joint left_gripper
- added joint JointLeftElbowFlex: type revolute, parent left_arm4_link, child left_arm5_link, origin xyz=0.145 0 0, axis 0 1 0, limit lower=-1.75 upper=1.75 effort=1.0 velocity=0.5
- added joint JointLeftForearmRoll: type revolute, parent left_arm5_link, child left_arm6_link, origin xyz=0.230643 0 0, axis 1 0 0, limit lower=-3.1415 upper=3.1415 effort=1.0 velocity=0.5
- added joint JointLeftGripper: type revolute, parent left_gripper1_link, child left_gripper2_link, origin xyz=0.024 -0.014 0 rpy=0 0 -1.5708, axis 0 0 1, limit lower=0 upper=1.5708 effort=1.0 velocity=0.5
- added joint JointLeftShoulderPan: type revolute, parent left_arm1_link, child left_arm2_link, origin xyz=0 0 -0.007, axis 0 0 1, limit lower=-1.5708 upper=1 effort=1.0 velocity=0.5
- added joint JointLeftShoulderTilt: type revolute, parent left_arm2_link, child left_arm3_link, origin xyz=0.139238 0 0, axis 0 1 0, limit lower=-1.5708 upper=1.5708 effort=1.0 velocity=0.5
- added joint JointLeftUpperArmRoll: type revolute, parent left_arm3_link, child left_arm4_link, origin xyz=0.238827 0 0, axis 1 0 0, limit lower=-3.1415 upper=3.1415 effort=1.0 velocity=0.5
- added joint JointLeftWristFlex: type revolute, parent left_arm6_link, child left_arm7_link, origin xyz=0.165 0 0, axis 0 1 0, limit lower=-1.75 upper=1.75 effort=1.0 velocity=0.5
- added joint JointLeftWristRoll: type revolute, parent left_arm7_link, child left_arm8_link, origin xyz=0.045311 0 0, axis 1 0 0, limit lower=-2 upper=2 effort=1.0 velocity=0.5
- joint left_gripper1_to_left_gripper3: mimic joint=left_gripper multiplier=-1 offset=0 -> joint=JointLeftGripper multiplier=-1 offset=0
- joint left_gripper1_to_left_gripper4l: mimic joint=left_gripper multiplier=-1 offset=0 -> joint=JointLeftGripper multiplier=-1 offset=0
- joint left_gripper1_to_left_gripper4r: mimic joint=left_gripper multiplier=1 offset=0 -> joint=JointLeftGripper multiplier=1 offset=0
- joint left_gripper2_to_left_gripper6: mimic joint=left_gripper multiplier=-1 offset=0 -> joint=JointLeftGripper multiplier=-1 offset=0
- joint left_gripper3_to_left_gripper5: mimic joint=left_gripper multiplier=1 offset=0 -> joint=JointLeftGripper multiplier=1 offset=0

Commit message: changed joint names

File: urdf/tr1.urdf (robot description, URDF)
Before this commit: robot tr1, 39 links, 38 joints
Joints:
- removed joint base_to_body
- removed joint base_to_wheel1
- removed joint base_to_wheel2
- removed joint base_to_wheel3
- removed joint base_to_wheel4
- added joint JointBaseWheelBL: type continuous, parent base_link, child wheel3_link, origin xyz=0.293310 -0.168810 -0.0725 rpy=0 0 -2.35619449019, axis 0 1 0
- added joint JointBaseWheelBR: type continuous, parent base_link, child wheel4_link, origin xyz=-0.293310 -0.168810 -0.0725 rpy=0 0 2.356194490191, axis 0 1 0
- added joint JointBaseWheelFL: type continuous, parent base_link, child wheel1_link, origin xyz=-0.293310 0.417810 -0.0725 rpy=0 0 0.785398, axis 0 1 0
- added joint JointBaseWheelFR: type continuous, parent base_link, child wheel2_link, origin xyz=0.293310 0.417810 -0.0725 rpy=0 0 -0.785398, axis 0 1 0
- added joint JointTorsoExtension: type prismatic, parent base_link, child body_link, origin xyz=0 0 0.7955, axis 0 0 1, limit lower=0 upper=0.300 effort=1000.0 velocity=0.0001
