Commit message: gazebo support

File: urdf/tr1.urdf (robot description, URDF)
Before this commit: robot tr1, 39 links, 38 joints
Links:
- link base_link: mass None -> 1.0; geometry collision mesh filename=package://tr1_description/meshes/dae/base.dae scale=0.001 0.001 0.001; visual mesh filename=package://tr1_description/meshes/dae/base.dae scale=0.001 0.001 0.001
- link body_link: mass None -> 1.0; geometry collision mesh filename=package://tr1_description/meshes/dae/body.dae scale=0.001 0.001 0.001; visual mesh filename=package://tr1_description/meshes/dae/body.dae scale=0.001 0.001 0.001
- link head_link: mass None -> 1.0; geometry collision mesh filename=package://tr1_description/meshes/dae/neck.dae scale=0.001 0.001 0.001; visual mesh filename=package://tr1_description/meshes/dae/head.dae scale=0.001 0.001 0.001
- link left_arm1_link: mass None -> 1.0; geometry collision mesh filename=package://tr1_description/meshes/dae/arm1.dae scale=0.001 0.001 0.001; visual mesh filename=package://tr1_description/meshes/dae/arm1.dae scale=0.001 0.001 0.001
- link left_arm2_link: mass None -> 1.0; geometry collision mesh filename=package://tr1_description/meshes/dae/arm2.dae scale=0.001 0.001 0.001; visual mesh filename=package://tr1_description/meshes/dae/arm2.dae scale=0.001 0.001 0.001
- link left_arm3_link: mass None -> 1.0; geometry collision mesh filename=package://tr1_description/meshes/dae/arm3.dae scale=0.001 0.001 0.001; visual mesh filename=package://tr1_description/meshes/dae/arm3.dae scale=0.001 0.001 0.001
- link left_arm4_link: mass None -> 1.0; geometry collision mesh filename=package://tr1_description/meshes/dae/arm4.dae scale=0.001 0.001 0.001; visual mesh filename=package://tr1_description/meshes/dae/arm4.dae scale=0.001 0.001 0.001
- link left_arm5_link: mass None -> 1.0; geometry collision mesh filename=package://tr1_description/meshes/dae/arm5.dae scale=0.001 0.001 0.001; visual mesh filename=package://tr1_description/meshes/dae/arm5.dae scale=0.001 0.001 0.001
- link left_arm6_link: mass None -> 1.0; geometry collision mesh filename=package://tr1_description/meshes/dae/arm6.dae scale=0.001 0.001 0.001; visual mesh filename=package://tr1_description/meshes/dae/arm6.dae scale=0.001 0.001 0.001
- link left_arm7_link: mass None -> 1.0; geometry collision mesh filename=package://tr1_description/meshes/dae/arm7.dae scale=0.001 0.001 0.001; visual mesh filename=package://tr1_description/meshes/dae/arm7.dae scale=0.001 0.001 0.001
- link left_arm8_link: mass None -> 1.0; geometry collision mesh filename=package://tr1_description/meshes/dae/arm8.dae scale=0.001 0.001 0.001; visual mesh filename=package://tr1_description/meshes/dae/arm8.dae scale=0.001 0.001 0.001
- link left_gripper1_link: mass None -> 1.0; geometry collision mesh filename=package://tr1_description/meshes/dae/gripper1.dae scale=0.001 0.001 0.001; visual mesh filename=package://tr1_description/meshes/dae/gripper1.dae scale=0.001 0.001 0.001
- link left_gripper2_link: mass None -> 1.0; geometry collision mesh filename=package://tr1_description/meshes/dae/gripper2.dae scale=0.001 0.001 0.001; visual mesh filename=package://tr1_description/meshes/dae/gripper2.dae scale=0.001 0.001 0.001
- link left_gripper3_link: mass None -> 1.0; geometry collision mesh filename=package://tr1_description/meshes/dae/gripper3.dae scale=0.001 0.001 0.001; visual mesh filename=package://tr1_description/meshes/dae/gripper3.dae scale=0.001 0.001 0.001
- link left_gripper4l_link: mass None -> 1.0; geometry collision mesh filename=package://tr1_description/meshes/dae/gripper4.dae scale=0.001 0.001 0.001; visual mesh filename=package://tr1_description/meshes/dae/gripper4.dae scale=0.001 0.001 0.001
- link left_gripper4r_link: mass None -> 1.0; geometry collision mesh filename=package://tr1_description/meshes/dae/gripper4.dae scale=0.001 0.001 0.001; visual mesh filename=package://tr1_description/meshes/dae/gripper4.dae scale=0.001 0.001 0.001
- link left_gripper5_link: mass None -> 1.0; geometry collision mesh filename=package://tr1_description/meshes/dae/gripper5.dae scale=0.001 0.001 0.001; visual mesh filename=package://tr1_description/meshes/dae/gripper5.dae scale=0.001 0.001 0.001
- link left_gripper6_link: mass None -> 1.0; geometry collision mesh filename=package://tr1_description/meshes/dae/gripper6.dae scale=0.001 0.001 0.001; visual mesh filename=package://tr1_description/meshes/dae/gripper6.dae scale=0.001 0.001 0.001
- link neck_base_link: mass None -> 1.0; geometry collision mesh filename=package://tr1_description/meshes/dae/neck_base.dae scale=0.001 0.001 0.001; visual mesh filename=package://tr1_description/meshes/dae/neck_base.dae scale=0.001 0.001 0.001
- link neck_link: mass None -> 1.0; geometry collision mesh filename=package://tr1_description/meshes/dae/neck.dae scale=0.001 0.001 0.001; visual mesh filename=package://tr1_description/meshes/dae/neck.dae scale=0.001 0.001 0.001
- link right_arm1_link: mass None -> 1.0; geometry collision mesh filename=package://tr1_description/meshes/dae/arm1.dae scale=0.001 0.001 0.001; visual mesh filename=package://tr1_description/meshes/dae/arm1.dae scale=0.001 0.001 0.001
- link right_arm2_link: mass None -> 1.0; geometry collision mesh filename=package://tr1_description/meshes/dae/arm2.dae scale=0.001 0.001 0.001; visual mesh filename=package://tr1_description/meshes/dae/arm2.dae scale=0.001 0.001 0.001
- link right_arm3_link: mass None -> 1.0; geometry collision mesh filename=package://tr1_description/meshes/dae/arm3.dae scale=0.001 0.001 0.001; visual mesh filename=package://tr1_description/meshes/dae/arm3.dae scale=0.001 0.001 0.001
- link right_arm4_link: mass None -> 1.0; geometry collision mesh filename=package://tr1_description/meshes/dae/arm4.dae scale=0.001 0.001 0.001; visual mesh filename=package://tr1_description/meshes/dae/arm4.dae scale=0.001 0.001 0.001
- link right_arm5_link: mass None -> 1.0; geometry collision mesh filename=package://tr1_description/meshes/dae/arm5.dae scale=0.001 0.001 0.001; visual mesh filename=package://tr1_description/meshes/dae/arm5.dae scale=0.001 0.001 0.001
- link right_arm6_link: mass None -> 1.0; geometry collision mesh filename=package://tr1_description/meshes/dae/arm6.dae scale=0.001 0.001 0.001; visual mesh filename=package://tr1_description/meshes/dae/arm6.dae scale=0.001 0.001 0.001
- link right_arm7_link: mass None -> 1.0; geometry collision mesh filename=package://tr1_description/meshes/dae/arm7.dae scale=0.001 0.001 0.001; visual mesh filename=package://tr1_description/meshes/dae/arm7.dae scale=0.001 0.001 0.001
- link right_arm8_link: mass None -> 1.0; geometry collision mesh filename=package://tr1_description/meshes/dae/arm8.dae scale=0.001 0.001 0.001; visual mesh filename=package://tr1_description/meshes/dae/arm8.dae scale=0.001 0.001 0.001
- link right_gripper1_link: mass None -> 1.0; geometry collision mesh filename=package://tr1_description/meshes/dae/gripper1.dae scale=0.001 0.001 0.001; visual mesh filename=package://tr1_description/meshes/dae/gripper1.dae scale=0.001 0.001 0.001
- link right_gripper2_link: mass None -> 1.0; geometry collision mesh filename=package://tr1_description/meshes/dae/gripper2.dae scale=0.001 0.001 0.001; visual mesh filename=package://tr1_description/meshes/dae/gripper2.dae scale=0.001 0.001 0.001
- link right_gripper3_link: mass None -> 1.0; geometry collision mesh filename=package://tr1_description/meshes/dae/gripper3.dae scale=0.001 0.001 0.001; visual mesh filename=package://tr1_description/meshes/dae/gripper3.dae scale=0.001 0.001 0.001
- link right_gripper4l_link: mass None -> 1.0; geometry collision mesh filename=package://tr1_description/meshes/dae/gripper4.dae scale=0.001 0.001 0.001; visual mesh filename=package://tr1_description/meshes/dae/gripper4.dae scale=0.001 0.001 0.001
- link right_gripper4r_link: mass None -> 1.0; geometry collision mesh filename=package://tr1_description/meshes/dae/gripper4.dae scale=0.001 0.001 0.001; visual mesh filename=package://tr1_description/meshes/dae/gripper4.dae scale=0.001 0.001 0.001
- link right_gripper5_link: mass None -> 1.0; geometry collision mesh filename=package://tr1_description/meshes/dae/gripper5.dae scale=0.001 0.001 0.001; visual mesh filename=package://tr1_description/meshes/dae/gripper5.dae scale=0.001 0.001 0.001
- link right_gripper6_link: mass None -> 1.0; geometry collision mesh filename=package://tr1_description/meshes/dae/gripper6.dae scale=0.001 0.001 0.001; visual mesh filename=package://tr1_description/meshes/dae/gripper6.dae scale=0.001 0.001 0.001
- link wheel1_link: mass None -> 1.0; geometry collision mesh filename=package://tr1_description/meshes/dae/wheel.dae scale=0.001 0.001 0.001; visual mesh filename=package://tr1_description/meshes/dae/wheel.dae scale=0.001 0.001 0.001
- link wheel2_link: mass None -> 1.0; geometry collision mesh filename=package://tr1_description/meshes/dae/wheel.dae scale=0.001 0.001 0.001; visual mesh filename=package://tr1_description/meshes/dae/wheel.dae scale=0.001 0.001 0.001
- link wheel3_link: mass None -> 1.0; geometry collision mesh filename=package://tr1_description/meshes/dae/wheel.dae scale=0.001 0.001 0.001; visual mesh filename=package://tr1_description/meshes/dae/wheel.dae scale=0.001 0.001 0.001
- link wheel4_link: mass None -> 1.0; geometry collision mesh filename=package://tr1_description/meshes/dae/wheel.dae scale=0.001 0.001 0.001; visual mesh filename=package://tr1_description/meshes/dae/wheel.dae scale=0.001 0.001 0.001
Joints:
- joint JointRightShoulderPan: limit lower=-1 upper=1.5708 effort=1.0 velocity=0.5 -> lower=-1 upper=1.5708 effort=1.0 velocity=0.1

Commit message: new head design

File: urdf/tr1.urdf (robot description, URDF)
Before this commit: robot tr1, 39 links, 38 joints
Links:
- link head_link: geometry collision mesh filename=package://tr1_description/meshes/dae/head.dae scale=0.1 0.1 0.1; visual mesh filename=package://tr1_description/meshes/dae/head.dae scale=0.1 0.1 0.1

Commit message: body design

File: urdf/tr1.urdf (robot description, URDF)
Before this commit: robot tr1, 39 links, 38 joints
Links:
- link body_link: geometry collision mesh filename=package://tr1_description/meshes/dae/body.dae scale=0.1 0.1 0.1; visual mesh filename=package://tr1_description/meshes/dae/body.dae scale=0.1 0.1 0.1
Joints:
- joint JointTorsoExtension: limit lower=0 upper=0.300 effort=1000.0 velocity=0.0001 -> lower=0 upper=0.150 effort=1000.0 velocity=0.0001; origin xyz=0 0 0.7955 -> xyz=0 0 0.7195

Commit message: torso and base alignment

File: urdf/tr1.urdf (robot description, URDF)
Before this commit: robot tr1, 39 links, 38 joints
Links:
- link base_link: geometry collision mesh filename=package://tr1_description/meshes/dae/base.dae scale=0.1 0.1 0.1; visual mesh filename=package://tr1_description/meshes/dae/base.dae scale=0.1 0.1 0.1
Joints:
- joint JointTorsoExtension: origin xyz=0 0 0.7195 -> xyz=0 0 0.707

Commit message: joint velocity and mass tuning

File: urdf/tr1.urdf (robot description, URDF)
Before this commit: robot tr1, 39 links, 38 joints
Links:
- link body_link: mass 1.0 -> 0.005
- link head_link: mass 1.0 -> 0.005
- link left_arm1_link: mass 1.0 -> 0.005
- link left_arm2_link: mass 1.0 -> 0.005
- link left_arm3_link: mass 1.0 -> 0.005
- link left_arm4_link: mass 1.0 -> 0.005
- link left_arm5_link: mass 1.0 -> 0.005
- link left_arm6_link: mass 1.0 -> 0.005
- link left_arm7_link: mass 1.0 -> 0.005
- link left_arm8_link: mass 1.0 -> 0.005
- link left_gripper1_link: mass 1.0 -> 0.005
- link left_gripper2_link: mass 1.0 -> 0.005
- link left_gripper3_link: mass 1.0 -> 0.005
- link left_gripper4l_link: mass 1.0 -> 0.005
- link left_gripper4r_link: mass 1.0 -> 0.005
- link left_gripper5_link: mass 1.0 -> 0.005
- link left_gripper6_link: mass 1.0 -> 0.005
- link neck_base_link: mass 1.0 -> 0.005
- link neck_link: mass 1.0 -> 0.005
- link right_arm1_link: mass 1.0 -> 0.005
- link right_arm2_link: mass 1.0 -> 0.005
- link right_arm3_link: mass 1.0 -> 0.005
- link right_arm4_link: mass 1.0 -> 0.005
- link right_arm5_link: mass 1.0 -> 0.005
- link right_arm6_link: mass 1.0 -> 0.005
- link right_arm7_link: mass 1.0 -> 0.005
- link right_arm8_link: mass 1.0 -> 0.005
- link right_gripper1_link: mass 1.0 -> 0.005
- link right_gripper2_link: mass 1.0 -> 0.005
- link right_gripper3_link: mass 1.0 -> 0.005
- link right_gripper4l_link: mass 1.0 -> 0.005
- link right_gripper4r_link: mass 1.0 -> 0.005
- link right_gripper5_link: mass 1.0 -> 0.005
- link right_gripper6_link: mass 1.0 -> 0.005
Joints:
- joint JointRightElbowFlex: limit lower=-1.75 upper=1.75 effort=1.0 velocity=0.5 -> lower=-1.75 upper=1.75 effort=1.0 velocity=0.1
- joint JointRightForearmRoll: limit lower=-3.1415 upper=3.1415 effort=1.0 velocity=0.5 -> lower=-3.1415 upper=3.1415 effort=1.0 velocity=1.4661
- joint JointRightShoulderPan: limit lower=-1 upper=1.5708 effort=1.0 velocity=0.1 -> lower=-1 upper=1.5708 effort=1.0 velocity=0.2932
- joint JointRightShoulderTilt: limit lower=-1.5708 upper=1.5708 effort=1.0 velocity=0.5 -> lower=-1.5708 upper=1.5708 effort=1.0 velocity=0.1
- joint JointRightUpperArmRoll: limit lower=-3.1415 upper=3.1415 effort=1.0 velocity=0.5 -> lower=-3.1415 upper=3.1415 effort=1.0 velocity=0.25
- joint JointRightWristFlex: limit lower=-1.75 upper=1.75 effort=1.0 velocity=0.5 -> lower=-1.75 upper=1.75 effort=1.0 velocity=0.7330
- joint JointRightWristRoll: limit lower=-2 upper=2 effort=1.0 velocity=0.5 -> lower=-2 upper=2 effort=1.0 velocity=7.5398

Commit message: urdf tuning

File: urdf/tr1.urdf (robot description, URDF)
Before this commit: robot tr1, 39 links, 38 joints
Joints:
- joint JointRightShoulderTilt: limit lower=-1.5708 upper=1.5708 effort=1.0 velocity=0.1 -> lower=-1.5708 upper=1.5708 effort=1.0 velocity=0.075

Commit message: coloring fix

File: urdf/tr1.urdf (robot description, URDF)
Before this commit: robot tr1, 39 links, 38 joints
Links:
- link base_link: geometry collision mesh filename=package://tr1_description/meshes/dae/base.dae scale=0.001 0.001 0.001; visual mesh filename=package://tr1_description/meshes/dae/base.dae scale=0.001 0.001 0.001
- link body_link: geometry collision mesh filename=package://tr1_description/meshes/dae/body.dae scale=0.001 0.001 0.001; visual mesh filename=package://tr1_description/meshes/dae/body.dae scale=0.001 0.001 0.001
- link head_link: geometry collision mesh filename=package://tr1_description/meshes/dae/head.dae scale=0.001 0.001 0.001; visual mesh filename=package://tr1_description/meshes/dae/head.dae scale=0.001 0.001 0.001
Joints:
- joint JointLeftElbowFlex: limit lower=-1.75 upper=1.75 effort=1.0 velocity=0.5 -> lower=-1.75 upper=1.75 effort=1.0 velocity=0.1
- joint JointLeftGripper: limit lower=0 upper=1.5708 effort=1.0 velocity=0.5 -> lower=0 upper=1.5708 effort=1.0 velocity=2.0
- joint JointLeftShoulderPan: limit lower=-1.5708 upper=1 effort=1.0 velocity=0.5 -> lower=-1.5708 upper=1 effort=1.0 velocity=1.5708
- joint JointLeftShoulderTilt: limit lower=-1.5708 upper=1.5708 effort=1.0 velocity=0.5 -> lower=-1.5708 upper=1.5708 effort=1.0 velocity=0.1
- joint JointLeftUpperArmRoll: limit lower=-3.1415 upper=3.1415 effort=1.0 velocity=0.5 -> lower=-3.1415 upper=3.1415 effort=1.0 velocity=0.25
- joint JointLeftWristFlex: limit lower=-1.75 upper=1.75 effort=1.0 velocity=0.5 -> lower=-1.75 upper=1.75 effort=1.0 velocity=0.7330
- joint JointLeftWristRoll: limit lower=-2 upper=2 effort=1.0 velocity=0.5 -> lower=-2 upper=2 effort=1.0 velocity=7.5398
